File: pcb/eflashy32.sch (KiCad schematic (older format))
At the start: 30 parts, among them J1 SERIAL, J2 10137062-00021LF, J3 SERIAL2, Q1 MMDT3904, SW1 JS202011CQN, U1 USBLC6-2SC6, U2 CP2102N-A02-GQFN24, U3 TLV75533PDBV

Commit message: prejig
Parts:
- C1: LCSC CERAMIC +/- 20% -> C28323
- C2, C9: LCSC CERAMIC +/- 20% -> C49678
- C5, C6: LCSC CERAMIC +/- 20% -> C1779
- D1, D2: LCSC C205441 -> C2293
- D3: LCSC C205442 -> C2297
- D4: value POWER -> PWR; LCSC C205444 -> C84256
- R1, R18, R2, R3: LCSC 1/8W, +/-5% -> C17414
- R15: LCSC 1/8W, +/-5% -> C17560
- R16: LCSC 1/8W, +/-5% -> C17713
- R17: value 1k -> 5k1; LCSC 1/8W, +/-5% -> C17513
- R4, R5: LCSC 1/8W, +/-5% -> C27834
- R6, R7: LCSC 1/8W, +/-5% -> C17513
- U3: LCSC C404027 -> C255621 C404027
Changed lines of the file:
@@
 F 2 "LED_SMD:LED_0805_2012Metric" H 7675 3550 50  0001 C CNN
 F 3 "~" H 7675 3550 50  0001 C CNN
-F 4 "C205441" V 7675 3550 50  0001 C CNN "LCSC"
+F 4 "C2293" V 7675 3550 50  0001 C CNN "LCSC"
 	1    7675 3550
 	0    -1   -1   0
@@
 F 2 "LED_SMD:LED_0805_2012Metric" H 8025 3550 50  0001 C CNN
 F 3 "" H 8025 3550 50  0001 C CNN
-F 4 "C205441" V 8025 3550 50  0001 C CNN "LCSC"
+F 4 "C2293" V 8025 3550 50  0001 C CNN "LCSC"
 	1    8025 3550
 	0    -1   -1   0
@@
 F 2 "Resistor_SMD:R_0805_2012Metric" H 8025 3300 50  0001 C CNN
 F 3 "~" H 8025 3300 50  0001 C CNN
-F 4 "1/8W, +/-5%" H 8025 3300 50  0001 C CNN "LCSC"
+F 4 "C17414" H 8025 3300 50  0001 C CNN "LCSC"
 	1    8025 3300
 	1    0    0    -1
@@
 F 2 "Resistor_SMD:R_0805_2012Metric" H 7675 3300 50  0001 C CNN
 F 3 "~" H 7675 3300 50  0001 C CNN
-F 4 "1/8W, +/-5%" H 7675 3300 50  0001 C CNN "LCSC"
+F 4 "C17414" H 7675 3300 50  0001 C CNN "LCSC"
 	1    7675 3300
 	1    0    0    -1
@@
 F 2 "Capacitor_SMD:C_0805_2012Metric" H 1900 1100 50  0001 C CNN
 F 3 "~" H 1900 1100 50  0001 C CNN
-F 4 "CERAMIC +/- 20%" H 1900 1100 50  0001 C CNN "LCSC"
+F 4 "C1779" H 1900 1100 50  0001 C CNN "LCSC"
 	1    1900 1100
 	1    0    0    -1
@@
 F 2 "Resistor_SMD:R_0805_2012Metric" H 5150 2650 50  0001 C CNN
 F 3 "~" H 5150 2650 50  0001 C CNN
-F 4 "1/8W, +/-5%" H 5150 2650 50  0001 C CNN "LCSC"
+F 4 "C17414" H 5150 2650 50  0001 C CNN "LCSC"
 	1    5150 2650
 	1    0    0    -1
@@
 F 2 "Capacitor_SMD:C_0805_2012Metric" H 3550 3300 50  0001 C CNN
 F 3 "~" H 3550 3300 50  0001 C CNN
-F 4 "CERAMIC +/- 20%" H 3550 3300 50  0001 C CNN "LCSC"
+F 4 "C49678" H 3550 3300 50  0001 C CNN "LCSC"
 	1    3550 3300
 	1    0    0    -1
@@
 F 2 "LED_SMD:LED_0805_2012Metric" H 8400 3550 50  0001 C CNN
 F 3 "~" H 8400 3550 50  0001 C CNN
-F 4 "C205442" V 8400 3550 50  0001 C CNN "LCSC"
+F 4 "C2297" V 8400 3550 50  0001 C CNN "LCSC"
 	1    8400 3550
 	0    -1   -1   0
@@
 P 8400 3300
 F 0 "R17" H 8459 3346 50  0000 L CNN
-F 1 "1k" H 8459 3255 50  0000 L CNN
+F 1 "5k1" H 8459 3255 50  0000 L CNN
 F 2 "Resistor_SMD:R_0805_2012Metric" H 8400 3300 50  0001 C CNN
 F 3 "~" H 8400 3300 50  0001 C CNN
-F 4 "1/8W, +/-5%" H 8400 3300 50  0001 C CNN "LCSC"
+F 4 "C17513" H 8400 3300 50  0001 C CNN "LCSC"
 	1    8400 3300
 	1    0    0    -1
@@
 P 8850 3550
 F 0 "D4" V 8889 3432 50  0000 R CNN
-F 1 "POWER" V 8798 3432 50  0000 R CNN
+F 1 "PWR" V 8798 3432 50  0000 R CNN
 F 2 "LED_SMD:LED_0805_2012Metric" H 8850 3550 50  0001 C CNN
 F 3 "~" H 8850 3550 50  0001 C CNN
-F 4 "C205444" V 8850 3550 50  0001 C CNN "LCSC"
+F 4 "C84256" V 8850 3550 50  0001 C CNN "LCSC"
 	1    8850 3550
 	0    -1   -1   0
@@
 F 2 "Resistor_SMD:R_0805_2012Metric" H 8850 3300 50  0001 C CNN
 F 3 "~" H 8850 3300 50  0001 C CNN
-F 4 "1/8W, +/-5%" H 8850 3300 50  0001 C CNN "LCSC"
+F 4 "C17414" H 8850 3300 50  0001 C CNN "LCSC"
 	1    8850 3300
 	1    0    0    -1
@@
 F 2 "Resistor_SMD:R_0805_2012Metric" H 4450 3650 50  0001 C CNN
 F 3 "~" H 4450 3650 50  0001 C CNN
-F 4 "1/8W, +/-5%" H 4450 3650 50  0001 C CNN "LCSC"
+F 4 "C17560" H 4450 3650 50  0001 C CNN "LCSC"
 	1    4450 3650
 	1    0    0    -1
@@
 F 2 "Resistor_SMD:R_0805_2012Metric" H 4450 3850 50  0001 C CNN
 F 3 "~" H 4450 3850 50  0001 C CNN
-F 4 "1/8W, +/-5%" H 4450 3850 50  0001 C CNN "LCSC"
+F 4 "C17713" H 4450 3850 50  0001 C CNN "LCSC"
 	1    4450 3850
 	1    0    0    -1
@@
 F 2 "Capacitor_SMD:C_0805_2012Metric" H 4650 2950 50  0001 C CNN
 F 3 "~" H 4650 2950 50  0001 C CNN
-F 4 "CERAMIC +/- 20%" H 4650 2950 50  0001 C CNN "LCSC"
+F 4 "C49678" H 4650 2950 50  0001 C CNN "LCSC"
 	1    4650 2950
 	1    0    0    -1
@@
 F 2 "Capacitor_SMD:C_0805_2012Metric" H 4250 2950 50  0001 C CNN
 F 3 "~" H 4250 2950 50  0001 C CNN
-F 4 "CERAMIC +/- 20%" H 4250 2950 50  0001 C CNN "LCSC"
+F 4 "C1779" H 4250 2950 50  0001 C CNN "LCSC"
 	1    4250 2950
 	1    0    0    -1
@@
 F 2 "Resistor_SMD:R_0805_2012Metric" H 5250 950 50  0001 C CNN
 F 3 "~" H 5250 950 50  0001 C CNN
-F 4 "1/8W, +/-5%" H 5250 950 50  0001 C CNN "LCSC"
+F 4 "C27834" H 5250 950 50  0001 C CNN "LCSC"
 	1    5250 950
 	0    1    1    0
@@
 F 2 "Resistor_SMD:R_0805_2012Metric" H 5250 1600 50  0001 C CNN
 F 3 "~" H 5250 1600 50  0001 C CNN
-F 4 "1/8W, +/-5%" H 5250 1600 50  0001 C CNN "LCSC"
+F 4 "C27834" H 5250 1600 50  0001 C CNN "LCSC"
 	1    5250 1600
 	0    1    1    0
@@
 F 2 "Resistor_SMD:R_0805_2012Metric" H 1750 4050 50  0001 C CNN
 F 3 "~" H 1750 4050 50  0001 C CNN
-F 4 "1/8W, +/-5%" H 1750 4050 50  0001 C CNN "LCSC"
+F 4 "C17513" H 1750 4050 50  0001 C CNN "LCSC"
 	1    1750 4050
 	1    0    0    -1
@@
 F 2 "Resistor_SMD:R_0805_2012Metric" H 2150 4050 50  0001 C CNN
 F 3 "~" H 2150 4050 50  0001 C CNN
-F 4 "1/8W, +/-5%" H 2150 4050 50  0001 C CNN "LCSC"
+F 4 "C17513" H 2150 4050 50  0001 C CNN "LCSC"
 	1    2150 4050
 	1    0    0    -1
@@
 F 2 "Capacitor_SMD:C_0805_2012Metric" H 1050 1100 50  0001 C CNN
 F 3 "~" H 1050 1100 50  0001 C CNN
-F 4 "CERAMIC +/- 20%" H 1050 1100 50  0001 C CNN "LCSC"
+F 4 "C28323" H 1050 1100 50  0001 C CNN "LCSC"
 	1    1050 1100
 	1    0    0    -1
@@
 F 2 "Package_TO_SOT_SMD:SOT-23-5" H 1500 1425 50  0001 C CIN
 F 3 "http://www.ti.com/lit/ds/symlink/tlv755p.pdf" H 1500 1150 50  0001 C CNN
-F 4 "C404027" H 1500 1100 50  0001 C CNN "LCSC"
+F 4 "C255621 C404027" H 1500 1100 50  0001 C CNN "LCSC"
 	1    1500 1100
 	1    0    0    -1

Commit message: change to 4 line
Parts:
- removed U1: USBLC6-2SC6, Package_TO_SOT_SMD:SOT-23-6, symbol Power_Protection:USBLC6-2SC6
- added U1: ESD PROTECTION, Package_TO_SOT_SMD:SOT-23-6, symbol Power_Protection:USBLC6-4SC6
Connections:
- net DOUT+ is gone; now on net DIN+: U2.3 (D+)
- net DOUT- is gone; now on net DIN-: U2.4 (D-)
- net DIN+: now also U1.1 (I/O1)
- net DIN-: now also U1.3 (I/O2)
- net GND: now also U1.2 (GND)
- net VBUS: now also U1.5 (VBUS)
- no-connect marks 12 -> 14
Changed lines of the file:
@@
 GPIO0
-$Comp
-L Power_Protection:USBLC6-2SC6 U1
-U 1 1 5F039FD8
-P 2750 3300
-F 0 "U1" H 2750 3881 50  0000 C CNN
-F 1 "USBLC6-2SC6" H 2750 3790 50  0000 C CNN
-F 2 "Package_TO_SOT_SMD:SOT-23-6" H 2750 2800 50  0001 C CNN
-F 3 "https://www.st.com/resource/en/datasheet/usblc6-2.pdf" H 2950 3650 50  0001 C CNN
-F 4 "C7519" H 2750 3300 50  0001 C CNN "LCSC"
-	1    2750 3300
-	1    0    0    -1
-$EndComp
 $Comp
 L power:GND #PWR05
@@
 Wire Wire Line
 	1650 3150 1750 3150
-Text Label 3150 3200 0    50   ~ 0
-DOUT-
-Text Label 2350 3400 2    50   ~ 0
-DIN+
-Text Label 2350 3200 2    50   ~ 0
-DOUT+
 $Comp
 L Device:C_Small C2
@@
 $EndComp
 Wire Wire Line
-	2750 2900 3550 2900
-Wire Wire Line
 	3550 2900 3550 3200
 Wire Wire Line
@@
 Wire Wire Line
 	3550 3700 2750 3700
-Connection ~ 2750 3700
 $Comp
 L Device:LED D3
@@
 Wire Wire Line
 	2050 2550 2050 2900
-Connection ~ 2750 2900
 Wire Wire Line
 	1950 2550 2050 2550
@@
 Text Label 1750 3350 0    50   ~ 0
 DIN+
-Text Label 3150 3400 0    50   ~ 0
-DIN-
 NoConn ~ 750  4050
 $Comp
@@
 	2250 2600 2250 2900
 Connection ~ 2250 2900
-Wire Wire Line
-	2250 2900 2750 2900
 NoConn ~ 1650 3650
 NoConn ~ 1650 3750
@@
 	1650 2150 1650 2550
 Connection ~ 1650 2550
+$Comp
+L Power_Protection:USBLC6-4SC6 U1
+U 1 1 5F1989DD
+P 2750 3300
+F 0 "U1" H 2750 3881 50  0000 C CNN
+F 1 "ESD PROTECTION" H 2750 3790 50  0000 C CNN
+F 2 "Package_TO_SOT_SMD:SOT-23-6" H 2750 2800 50  0001 C CNN
+F 3 "https://www.st.com/resource/en/datasheet/usblc6-4.pdf" H 2950 3650 50  0001 C CNN
+F 4 "C294963" H 2750 3300 50  0001 C CNN "LCSC"
+	1    2750 3300
+	1    0    0    -1
+$EndComp
+Text Label 2350 3200 2    50   ~ 0
+DIN+
+Text Label 2350 3050 2    50   ~ 0
+DOUT+
+Wire Wire Line
+	2350 3200 2350 3050
+Text Label 2350 3400 2    50   ~ 0
+DIN-
+Text Label 2350 3500 2    50   ~ 0
+DOUT-
+Wire Wire Line
+	2250 2900 2750 2900
+Connection ~ 2750 2900
+Wire Wire Line
+	2750 2900 3550 2900
+Connection ~ 2750 3700
+Wire Wire Line
+	2350 3500 2350 3400
+NoConn ~ 3150 3200
+NoConn ~ 3150 3400
 $EndSCHEMATC

Commit message: docs
Parts:
- R1, R18, R2: value 1k -> 10k
- R17: value 5k1 -> 10k; LCSC C17513 -> C17414
- R3: LCSC C17414 -> C17513
- R4, R5: LCSC C27834 -> C17414
- R6, R7: LCSC C17513 -> C27834
Changed lines of the file:
@@
 P 8025 3300
 F 0 "R2" H 8084 3346 50  0000 L CNN
-F 1 "1k" H 8084 3255 50  0000 L CNN
+F 1 "10k" H 8084 3255 50  0000 L CNN
 F 2 "Resistor_SMD:R_0805_2012Metric" H 8025 3300 50  0001 C CNN
 F 3 "~" H 8025 3300 50  0001 C CNN
@@
 P 7675 3300
 F 0 "R1" H 7734 3346 50  0000 L CNN
-F 1 "1k" H 7734 3255 50  0000 L CNN
+F 1 "10k" H 7734 3255 50  0000 L CNN
 F 2 "Resistor_SMD:R_0805_2012Metric" H 7675 3300 50  0001 C CNN
 F 3 "~" H 7675 3300 50  0001 C CNN
@@
 F 2 "Resistor_SMD:R_0805_2012Metric" H 5150 2650 50  0001 C CNN
 F 3 "~" H 5150 2650 50  0001 C CNN
-F 4 "C17414" H 5150 2650 50  0001 C CNN "LCSC"
+F 4 "C17513" H 5150 2650 50  0001 C CNN "LCSC"
 	1    5150 2650
 	1    0    0    -1
@@
 P 8400 3300
 F 0 "R17" H 8459 3346 50  0000 L CNN
-F 1 "5k1" H 8459 3255 50  0000 L CNN
+F 1 "10k" H 8459 3255 50  0000 L CNN
 F 2 "Resistor_SMD:R_0805_2012Metric" H 8400 3300 50  0001 C CNN
 F 3 "~" H 8400 3300 50  0001 C CNN
-F 4 "C17513" H 8400 3300 50  0001 C CNN "LCSC"
+F 4 "C17414" H 8400 3300 50  0001 C CNN "LCSC"
 	1    8400 3300
 	1    0    0    -1
@@
 P 8850 3300
 F 0 "R18" H 8909 3346 50  0000 L CNN
-F 1 "1k" H 8909 3255 50  0000 L CNN
+F 1 "10k" H 8909 3255 50  0000 L CNN
 F 2 "Resistor_SMD:R_0805_2012Metric" H 8850 3300 50  0001 C CNN
 F 3 "~" H 8850 3300 50  0001 C CNN
@@
 F 2 "Resistor_SMD:R_0805_2012Metric" H 5250 950 50  0001 C CNN
 F 3 "~" H 5250 950 50  0001 C CNN
-F 4 "C27834" H 5250 950 50  0001 C CNN "LCSC"
+F 4 "C17414" H 5250 950 50  0001 C CNN "LCSC"
 	1    5250 950
 	0    1    1    0
@@
 F 2 "Resistor_SMD:R_0805_2012Metric" H 5250 1600 50  0001 C CNN
 F 3 "~" H 5250 1600 50  0001 C CNN
-F 4 "C27834" H 5250 1600 50  0001 C CNN "LCSC"
+F 4 "C17414" H 5250 1600 50  0001 C CNN "LCSC"
 	1    5250 1600
 	0    1    1    0
@@
 F 2 "Resistor_SMD:R_0805_2012Metric" H 1750 4050 50  0001 C CNN
 F 3 "~" H 1750 4050 50  0001 C CNN
-F 4 "C17513" H 1750 4050 50  0001 C CNN "LCSC"
+F 4 "C27834" H 1750 4050 50  0001 C CNN "LCSC"
 	1    1750 4050
 	1    0    0    -1
@@
 F 2 "Resistor_SMD:R_0805_2012Metric" H 2150 4050 50  0001 C CNN
 F 3 "~" H 2150 4050 50  0001 C CNN
-F 4 "C17513" H 2150 4050 50  0001 C CNN "LCSC"
+F 4 "C27834" H 2150 4050 50  0001 C CNN "LCSC"
 	1    2150 4050
 	1    0    0    -1

Commit message: update
Parts:
- J2: symbol Connector:USB_C_Receptacle_USB2.0 -> eflashy32-rescue:USB_C_Receptacle_USB2.0-Connector; LCSC DNP -> C388659
- U2: symbol Interface_USB:CP2102N-A01-GQFN24 -> eflashy32-rescue:CP2102N-A01-GQFN24-Interface_USB; LCSC ??? -> C969151
Changed lines of the file:
@@
 NoConn ~ 750  4050
 $Comp
-L Interface_USB:CP2102N-A01-GQFN24 U2
+L eflashy32-rescue:CP2102N-A01-GQFN24-Interface_USB U2
 U 1 1 5EFF7E9C
 P 5900 3350
@@
 F 2 "Package_DFN_QFN:QFN-24-1EP_4x4mm_P0.5mm_EP2.6x2.6mm" H 6350 2550 50  0001 L CNN
 F 3 "https://www.silabs.com/documents/public/data-sheets/cp2102n-datasheet.pdf" H 5950 2300 50  0001 C CNN
-F 4 "???" H 5900 3350 50  0001 C CNN "LCSC"
+F 4 "C969151" H 5900 3350 50  0001 C CNN "LCSC"
 	1    5900 3350
 	1    0    0    -1
@@
 Connection ~ 1650 3150
 $Comp
-L Connector:USB_C_Receptacle_USB2.0 J2
+L eflashy32-rescue:USB_C_Receptacle_USB2.0-Connector J2
 U 1 1 5F25798E
 P 1050 3150
@@
 F 2 "!Greg:USBC-Amphenol-10137062-00021LF" H 1200 3150 50  0001 C CNN
 F 3 "https://www.usb.org/sites/default/files/documents/usb_type-c.zip" H 1200 3150 50  0001 C CNN
-F 4 "DNP" H 1050 3150 50  0001 C CNN "LCSC"
+F 4 "C388659" H 1050 3150 50  0001 C CNN "LCSC"
 	1    1050 3150
 	1    0    0    -1
